Commit message: implementation finished, ready for test

File: my_robot/urdf/my_robot.xacro (robot description, xacro)
@@ -34,5 +34,5 @@
       <origin xyz="-0.15 0 -0.1" rpy=" 0 0 0"/>
       <geometry>
-        <sphere radius="0.048"/>
+        <sphere radius="0.04"/>
       </geometry>
     </collision>
@@ -52,5 +52,5 @@
       <origin xyz="0.15 0 -0.1" rpy=" 0 0 0"/>
       <geometry>
-        <sphere radius="0.0499"/>
+        <sphere radius="0.05"/>
       </geometry>
     </visual>
